File: CanSwitch/CanSwitch.sch (EAGLE design)
At the start: 17 parts

Commit message: cleanup after renaming libraries earlier this year and dropping auto routed nets in board to start from scratch again
Parts:
- RJ45CONNECTOR: device GME:WEBP88GME -> PoJD:WEBP88GME
- SWITCHINPUT: device GME:PTRAK700250GME -> PoJD:PTRAK700250GME
Changed lines of the file:
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@@
 <part name="CHIP" library="microchip" deviceset="PIC18F2*80" device="-I/SP" technology="4"/>
 <part name="DEBUGGING" library="pinhead" deviceset="PINHD-1X5" device=""/>
-<part name="RJ45CONNECTOR" library="GME" deviceset="WEBP88" device="GME"/>
-<part name="SWITCHINPUT" library="GME" deviceset="PTRAK700250" device="GME"/>
+<part name="RJ45CONNECTOR" library="PoJD" deviceset="WEBP88" device="GME"/>
+<part name="SWITCHINPUT" library="PoJD" deviceset="PTRAK700250" device="GME"/>
 <part name="MCP2561" library="PoJD" deviceset="MCP2561" device="MCP"/>
 <part name="MCLR_J" library="jumper" deviceset="JP1Q" device=""/>
