File: CanSwitch/CanSwitch.sch (EAGLE design)
At the start: 17 parts

Commit message: swapped proper package for capacitor and also updated library components and little tweaks to the wires
Parts:
- C1, C2, C3, C7, CXT1, CXT2: device rcl:C-EUC0805 -> rcl:C-EU025-025X050
Changed lines of the file:
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@@
 <part name="GND2" library="supply1" deviceset="GND" device=""/>
 <part name="P+2" library="supply1" deviceset="+5V" device=""/>
-<part name="C1" library="rcl" deviceset="C-EU" device="C0805" value="0.1uF"/>
+<part name="C1" library="rcl" deviceset="C-EU" device="025-025X050" value="0.1uF"/>
 <part name="GND4" library="supply1" deviceset="GND" device=""/>
 <part name="P+3" library="supply1" deviceset="+5V" device=""/>
-<part name="C2" library="rcl" deviceset="C-EU" device="C0805" value="0.1uF"/>
-<part name="C7" library="rcl" deviceset="C-EU" device="C0805" value="10 uF"/>
+<part name="C2" library="rcl" deviceset="C-EU" device="025-025X050" value="0.1uF"/>
+<part name="C7" library="rcl" deviceset="C-EU" device="025-025X050" value="10 uF"/>
 <part name="GND5" library="supply1" deviceset="GND" device=""/>
-<part name="CXT1" library="rcl" deviceset="C-EU" device="C0805" value="33pF"/>
-<part name="CXT2" library="rcl" deviceset="C-EU" device="C0805" value="33pF"/>
+<part name="CXT1" library="rcl" deviceset="C-EU" device="025-025X050" value="33pF"/>
+<part name="CXT2" library="rcl" deviceset="C-EU" device="025-025X050" value="33pF"/>
 <part name="GND6" library="supply1" deviceset="GND" device=""/>
 <part name="R3" library="rcl" deviceset="R-EU_" device="0207/10" value="1kOhm"/>
@@
 <part name="P+1" library="supply1" deviceset="+5V" device=""/>
 <part name="GND3" library="supply1" deviceset="GND" device=""/>
-<part name="C3" library="rcl" deviceset="C-EU" device="C0805" value="0.1uF"/>
+<part name="C3" library="rcl" deviceset="C-EU" device="025-025X050" value="0.1uF"/>
 <part name="XTAL" library="special" deviceset="XTAL/S" device="" value="16MHz"/>
 </parts>

Commit message: #2 renamed few components, moved all to new origin, added holes for final drilling, added silkcreen to desc all, including signature. Not to print out names layers, only place and values layers in the final silkscreen
Parts:
- R1: value 10kOhm -> 10000
- R2: value 470Ohm -> 470
- R3: value 1kOhm -> 1000
Changed lines of the file:
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@@
 <part name="MCP2561" library="PoJD" deviceset="MCP2561" device="MCP"/>
 <part name="MCLR_J" library="jumper" deviceset="JP1Q" device=""/>
-<part name="R1" library="rcl" deviceset="R-EU_" device="0207/10" value="10kOhm"/>
-<part name="R2" library="rcl" deviceset="R-EU_" device="0207/10" value="470Ohm"/>
+<part name="R1" library="rcl" deviceset="R-EU_" device="0207/10" value="10000"/>
+<part name="R2" library="rcl" deviceset="R-EU_" device="0207/10" value="470"/>
 <part name="GND2" library="supply1" deviceset="GND" device=""/>
 <part name="P+2" library="supply1" deviceset="+5V" device=""/>
@@
 <part name="CXT2" library="rcl" deviceset="C-EU" device="025-025X050" value="33pF"/>
 <part name="GND6" library="supply1" deviceset="GND" device=""/>
-<part name="R3" library="rcl" deviceset="R-EU_" device="0207/10" value="1kOhm"/>
+<part name="R3" library="rcl" deviceset="R-EU_" device="0207/10" value="1000"/>
 <part name="STATUSLED" library="led" deviceset="LED" device="5MM"/>
 <part name="GND7" library="supply1" deviceset="GND" device=""/>

Commit message: #5 new component for RJ45 WEBPP single, also renamed old one to DOUBLE and updated CanSwitch project references, used in CanRelay now and added all the wiring to it too
Parts:
- RJ45CONNECTOR: value WEBP88GME -> WEBP88_DDOUBLE; device PoJD:WEBP88GME -> PoJD:WEBP88_DDOUBLE
Changed lines of the file:
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@@
 <part name="CHIP" library="microchip" deviceset="PIC18F2*80" device="-I/SP" technology="4"/>
 <part name="DEBUGGING" library="pinhead" deviceset="PINHD-1X5" device=""/>
-<part name="RJ45CONNECTOR" library="PoJD" deviceset="WEBP88" device="GME"/>
+<part name="RJ45CONNECTOR" library="PoJD" deviceset="WEBP88_D" device="DOUBLE"/>
 <part name="SWITCHINPUT" library="PoJD" deviceset="PTRAK700250" device="GME"/>
 <part name="MCP2561" library="PoJD" deviceset="MCP2561" device="MCP"/>

Commit message: final tuning of both boards - squeezing switch board a bit yet, adding some more silkscreen, exporting to image to share on some electrical forums for checks
Connections:
- net N$3 renamed OSC2
- net N$6 renamed OSC1
Changed lines of the file:
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@@
 </segment>
 </net>
-<net name="N$6" class="0">
+<net name="OSC1" class="0">
 <segment>
 <pinref part="CHIP" gate="G$1" pin="RA7/CLKI/OSC1"/>
@@
 </segment>
 </net>
-<net name="N$3" class="0">
+<net name="OSC2" class="0">
 <segment>
 <pinref part="CHIP" gate="G$1" pin="RA6/CLKO/OSC2"/>

Commit message: incorporated hints from web: set proper sizes for caps, left enough space for them to be bend on the board. Reviewed any acute angles in traces. Increased isolation in ground copper so that no so called GND fingers are in the PCB Relay board. Also double checked other footprints, XTAL is a bit larger than real, but not by much
Parts:
- C2, C3, C7: device rcl:C-EU025-025X050 -> rcl:C-EU050-025X075
- CXT1, CXT2: device rcl:C-EU025-025X050 -> rcl:C-EU025-030X050
Changed lines of the file:
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@@
 <grid distance="0.1" unitdist="inch" unit="inch" style="lines" multiple="1" display="no" altdistance="0.01" altunitdist="inch" altunit="inch"/>
 <layers>
-<layer number="1" name="Top" color="4" fill="1" visible="no" active="no"/>
-<layer number="16" name="Bottom" color="1" fill="1" visible="no" active="no"/>
-<layer number="17" name="Pads" color="2" fill="1" visible="no" active="no"/>
-<layer number="18" name="Vias" color="2" fill="1" visible="no" active="no"/>
-<layer number="19" name="Unrouted" color="6" fill="1" visible="no" active="no"/>
-<layer number="20" name="Dimension" color="15" fill="1" visible="no" active="no"/>
-<layer number="21" name="tPlace" color="7" fill="1" visible="no" active="no"/>
-<layer number="22" name="bPlace" color="7" fill="1" visible="no" active="no"/>
-<layer number="23" name="tOrigins" color="15" fill="1" visible="no" active="no"/>
-<layer number="24" name="bOrigins" color="15" fill="1" visible="no" active="no"/>
-<layer number="25" name="tNames" color="7" fill="1" visible="no" active="no"/>
-<layer number="26" name="bNames" color="7" fill="1" visible="no" active="no"/>
-<layer number="27" name="tValues" color="7" fill="1" visible="no" active="no"/>
-<layer number="28" name="bValues" color="7" fill="1" visible="no" active="no"/>
+<layer number="1" name="Top" color="4" fill="1" visible="yes" active="no"/>
+<layer number="16" name="Bottom" color="1" fill="1" visible="yes" active="no"/>
+<layer number="17" name="Pads" color="2" fill="1" visible="yes" active="no"/>
+<layer number="18" name="Vias" color="2" fill="1" visible="yes" active="no"/>
+<layer number="19" name="Unrouted" color="6" fill="1" visible="yes" active="no"/>
+<layer number="20" name="Dimension" color="15" fill="1" visible="yes" active="no"/>
+<layer number="21" name="tPlace" color="7" fill="1" visible="yes" active="no"/>
+<layer number="22" name="bPlace" color="7" fill="1" visible="yes" active="no"/>
+<layer number="23" name="tOrigins" color="15" fill="1" visible="yes" active="no"/>
+<layer number="24" name="bOrigins" color="15" fill="1" visible="yes" active="no"/>
+<layer number="25" name="tNames" color="7" fill="1" visible="yes" active="no"/>
+<layer number="26" name="bNames" color="7" fill="1" visible="yes" active="no"/>
+<layer number="27" name="tValues" color="7" fill="1" visible="yes" active="no"/>
+<layer number="28" name="bValues" color="7" fill="1" visible="yes" active="no"/>
 <layer number="29" name="tStop" color="7" fill="3" visible="no" active="no"/>
 <layer number="30" name="bStop" color="7" fill="6" visible="no" active="no"/>
@@
 <layer number="35" name="tGlue" color="7" fill="4" visible="no" active="no"/>
 <layer number="36" name="bGlue" color="7" fill="5" visible="no" active="no"/>
-<layer number="37" name="tTest" color="7" fill="1" visible="no" active="no"/>
-<layer number="38" name="bTest" color="7" fill="1" visible="no" active="no"/>
+<layer number="37" name="tTest" color="7" fill="1" visible="yes" active="no"/>
+<layer number="38" name="bTest" color="7" fill="1" visible="yes" active="no"/>
 <layer number="39" name="tKeepout" color="4" fill="11" visible="no" active="no"/>
 <layer number="40" name="bKeepout" color="1" fill="11" visible="no" active="no"/>
@@
 <layer number="44" name="Drills" color="7" fill="1" visible="no" active="no"/>
 <layer number="45" name="Holes" color="7" fill="1" visible="no" active="no"/>
-<layer number="46" name="Milling" color="3" fill="1" visible="no" active="no"/>
-<layer number="47" name="Measures" color="7" fill="1" visible="no" active="no"/>
-<layer number="48" name="Document" color="7" fill="1" visible="no" active="no"/>
-<layer number="49" name="Reference" color="7" fill="1" visible="no" active="no"/>
-<layer number="51" name="tDocu" color="7" fill="1" visible="no" active="no"/>
-<layer number="52" name="bDocu" color="7" fill="1" visible="no" active="no"/>
+<layer number="46" name="Milling" color="3" fill="1" visible="yes" active="no"/>
+<layer number="47" name="Measures" color="7" fill="1" visible="yes" active="no"/>
+<layer number="48" name="Document" color="7" fill="1" visible="yes" active="no"/>
+<layer number="49" name="Reference" color="7" fill="1" visible="yes" active="no"/>
+<layer number="51" name="tDocu" color="7" fill="1" visible="yes" active="no"/>
+<layer number="52" name="bDocu" color="7" fill="1" visible="yes" active="no"/>
 <layer number="90" name="Modules" color="5" fill="1" visible="yes" active="yes"/>
 <layer number="91" name="Nets" color="2" fill="1" visible="yes" active="yes"/>
@@
 <part name="GND4" library="supply1" deviceset="GND" device=""/>
 <part name="P+3" library="supply1" deviceset="+5V" device=""/>
-<part name="C2" library="rcl" deviceset="C-EU" device="025-025X050" value="0.1uF"/>
-<part name="C7" library="rcl" deviceset="C-EU" device="025-025X050" value="10 uF"/>
+<part name="C2" library="rcl" deviceset="C-EU" device="050-025X075" value="0.1uF"/>
+<part name="C7" library="rcl" deviceset="C-EU" device="050-025X075" value="10 uF"/>
 <part name="GND5" library="supply1" deviceset="GND" device=""/>
-<part name="CXT1" library="rcl" deviceset="C-EU" device="025-025X050" value="33pF"/>
-<part name="CXT2" library="rcl" deviceset="C-EU" device="025-025X050" value="33pF"/>
+<part name="CXT1" library="rcl" deviceset="C-EU" device="025-030X050" value="33pF"/>
+<part name="CXT2" library="rcl" deviceset="C-EU" device="025-030X050" value="33pF"/>
 <part name="GND6" library="supply1" deviceset="GND" device=""/>
 <part name="R3" library="rcl" deviceset="R-EU_" device="0207/10" value="1000"/>
@@
 <part name="P+1" library="supply1" deviceset="+5V" device=""/>
 <part name="GND3" library="supply1" deviceset="GND" device=""/>
-<part name="C3" library="rcl" deviceset="C-EU" device="025-025X050" value="0.1uF"/>
+<part name="C3" library="rcl" deviceset="C-EU" device="050-025X075" value="0.1uF"/>
 <part name="XTAL" library="special" deviceset="XTAL/S" device="" value="16MHz"/>
 </parts>
